File: MCUPower.kicad_sch (KiCad schematic)
At the start: 24 parts, among them J6 XT60, SW1 SW_SPST, SW2 SW_DIP_x02, U3 lm3940 LDO, U5 STM32F103C8Tx, Y2 abracon abm3 8mhz

Commit message: Add files via upload
Parts:
- R1: value 220 , 0603 -> 560 , 0603
- R2, R4: value 10k 0603 -> 4.7k 0603
Connections:
- net +3.3V: now also C17.1, C18.1, C26.1, C27.1, C29.1, C30.1, C31.1, R2.1, R4.2; no longer SW2.1, SW2.2
- net +5V: now also C15.1, C19.1, SW1.2 (B), U3.2 (VI)
- net BOOT0: now also SW2.4
- net BOOT1: now also R4.1, SW2.3; no longer R4.2
- net GND: now also SW2.1, SW2.2
- net USBDM renamed USBDN
Other:
- moved on the sheet: R2, R4, SW2
