File: peripherals.kicad_sch (KiCad schematic)
At the start: 27 parts, among them J8 Conn_01x04_Socket, J9 Conn_01x04_Socket, U6 BMP280 (Barometer), U7 MPU-6050 (IMU), U8 NEO-M9N

Commit message: Add files via upload
Parts:
- added D9: BAR_LED, LED_SMD:LED_0201_0603Metric, symbol Device:LED
- added R24: 220 , 0603, Resistor_SMD:R_0201_0603Metric, symbol Device:R
- AE1: footprint RF_Antenna:Antenova_SR4G013_GPS -> Connector_Coaxial:SMA_Amphenol_132134-11_Vertical
Connections:
- net +3.3V: now also R24.1
- net GND: now also D9.1 (K)
- new net: D9.2 (A), R24.2
Changed lines of the file:
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@@
   (junction (at 93.98 115.57) (diameter 0) (color 0 0 0 0)
+  )
+  (junction (at 76.2 34.29) (diameter 0) (color 0 0 0 0)
   )
   (junction (at 194.31 48.26) (diameter 0) (color 0 0 0 0)
@@
     (stroke (width 0) (type default))
   )
+  (wire (pts (xy 76.2 44.45) (xy 76.2 48.26))
+    (stroke (width 0) (type default))
+  )
   (wire (pts (xy 173.99 88.9) (xy 166.37 88.9))
     (stroke (width 0) (type default))
   )
+  (wire (pts (xy 83.82 34.29) (xy 87.63 34.29))
+    (stroke (width 0) (type default))
+  )
   (wire (pts (xy 214.63 132.08) (xy 215.9 132.08))
     (stroke (width 0) (type default))
@@
     (stroke (width 0) (type default))
   )
-  (wire (pts (xy 76.2 33.02) (xy 76.2 44.45))
-    (stroke (width 0) (type default))
-  )
-  (wire (pts (xy 76.2 44.45) (xy 76.2 48.26))
+  (wire (pts (xy 76.2 24.13) (xy 76.2 34.29))
+    (stroke (width 0) (type default))
+  )
+  (wire (pts (xy 76.2 34.29) (xy 76.2 44.45))
     (stroke (width 0) (type default))
   )
@@
       (effects (font (size 1.27 1.27)) (justify left))
     )
-    (property "Footprint" "RF_Antenna:Antenova_SR4G013_GPS" (at 215.9 118.745 0)
+    (property "Footprint" "Connector_Coaxial:SMA_Amphenol_132134-11_Vertical" (at 215.9 118.745 0)
       (effects (font (size 1.27 1.27)) hide)
     )
@@
     )
   )
+  (symbol (lib_id "Device:LED") (at 87.63 38.1 90) (unit 1)
+    (in_bom yes) (on_board yes) (dnp no) (fields_autoplaced)
+    (property "Reference" "D9" (at 91.44 38.4175 90)
+      (effects (font (size 1.27 1.27)) (justify right))
+    )
+    (property "Value" "BAR_LED" (at 91.44 40.9575 90)
+      (effects (font (size 1.27 1.27)) (justify right))
+    )
+    (property "Footprint" "LED_SMD:LED_0201_0603Metric" (at 87.63 38.1 0)
+      (effects (font (size 1.27 1.27)) hide)
+    )
+    (property "Datasheet" "~" (at 87.63 38.1 0)
+      (effects (font (size 1.27 1.27)) hide)
+    )
+    (pin "2")
+    (pin "1")
+    (instances
+      (project "Flightcontroller"
+        (path "/18c01021-77ec-4d91-95d9-b43bc6ef621c/8d94fec5-c0cd-4dcb-8d08-fa8de3169f79"
+          (reference "D9") (unit 1)
+        )
+      )
+    )
+  )
   (symbol (lib_id "power:GND") (at 207.01 104.14 0) (unit 1)
     (in_bom yes) (on_board yes) (dnp no) (fields_autoplaced)
@@
     )
   )
+  (symbol (lib_id "Device:R") (at 80.01 34.29 90) (unit 1)
+    (in_bom yes) (on_board yes) (dnp no) (fields_autoplaced)
+    (property "Reference" "R24" (at 80.01 27.94 90)
+      (effects (font (size 1.27 1.27)))
+    )
+    (property "Value" "220 , 0603" (at 80.01 30.48 90)
+      (effects (font (size 1.27 1.27)))
+    )
+    (property "Footprint" "Resistor_SMD:R_0201_0603Metric" (at 80.01 36.068 90)
+      (effects (font (size 1.27 1.27)) hide)
+    )
+    (property "Datasheet" "~" (at 80.01 34.29 0)
+      (effects (font (size 1.27 1.27)) hide)
+    )
+    (pin "1")
+    (pin "2")
+    (instances
+      (project "Flightcontroller"
+        (path "/18c01021-77ec-4d91-95d9-b43bc6ef621c/8d94fec5-c0cd-4dcb-8d08-fa8de3169f79"
+          (reference "R24") (unit 1)
+        )
+      )
+    )
+  )
   (symbol (lib_id "power:GND") (at 191.77 83.82 0) (unit 1)
     (in_bom yes) (on_board yes) (dnp no) (fields_autoplaced)
@@
     )
   )
-  (symbol (lib_id "power:+3.3V") (at 76.2 33.02 0) (unit 1)
-    (in_bom yes) (on_board yes) (dnp no) (fields_autoplaced)
-    (property "Reference" "#PWR059" (at 76.2 36.83 0)
-      (effects (font (size 1.27 1.27)) hide)
-    )
-    (property "Value" "+3.3V" (at 76.2 27.94 0)
-      (effects (font (size 1.27 1.27)))
-    )
-    (property "Footprint" "" (at 76.2 33.02 0)
-      (effects (font (size 1.27 1.27)) hide)
-    )
-    (property "Datasheet" "" (at 76.2 33.02 0)
+  (symbol (lib_id "power:+3.3V") (at 76.2 24.13 0) (unit 1)
+    (in_bom yes) (on_board yes) (dnp no) (fields_autoplaced)
+    (property "Reference" "#PWR059" (at 76.2 27.94 0)
+      (effects (font (size 1.27 1.27)) hide)
+    )
+    (property "Value" "+3.3V" (at 76.2 19.05 0)
+      (effects (font (size 1.27 1.27)))
+    )
+    (property "Footprint" "" (at 76.2 24.13 0)
+      (effects (font (size 1.27 1.27)) hide)
+    )
+    (property "Datasheet" "" (at 76.2 24.13 0)
       (effects (font (size 1.27 1.27)) hide)
     )
@@
         )
       )
+    )
+  )
+  (symbol (lib_id "power:GND") (at 87.63 41.91 0) (unit 1)
+    (in_bom yes) (on_board yes) (dnp no) (fields_autoplaced)
+    (property "Reference" "#PWR010" (at 87.63 48.26 0)
+      (effects (font (size 1.27 1.27)) hide)
+    )
+    (property "Value" "GND" (at 87.63 46.99 0)
+      (effects (font (size 1.27 1.27)))
+    )
+    (property "Footprint" "" (at 87.63 41.91 0)
+      (effects (font (size 1.27 1.27)) hide)
+    )
+    (property "Datasheet" "" (at 87.63 41.91 0)
+      (effects (font (size 1.27 1.27)) hide)
+    )
+    (pin "1")
+    (instances
+      (project "Flightcontroller"
+        (path "/18c01021-77ec-4d91-95d9-b43bc6ef621c/8d94fec5-c0cd-4dcb-8d08-fa8de3169f79"
+          (reference "#PWR010") (unit 1)
+        )
+      )
